Commit message: Add exploration env

File: urdf/jackal_velodyne.urdf.xacro (robot description, xacro)
@@ -171,5 +171,5 @@
        of these into the final description is controlled by optenv variables, which
        default each one to off.-->
-  <xacro:include filename="$(find jackal_description)/urdf/accessories.urdf.xacro" />
+  <!-- <xacro:include filename="$(find jackal_description)/urdf/accessories.urdf.xacro" /> -->
   <!-- Optional custom includes. -->
   <xacro:if value="$(optenv JACKAL_URDF_EXTRAS 0)">
@@ -178,6 +178,6 @@
   <!-- VLP-16 -->
   <xacro:include filename="$(find velodyne_description)/urdf/VLP-16.urdf.xacro"/>
-  <VLP-16 parent="base_link" name="velodyne" topic="/velodyne_points" hz="10" samples="180">
-    <origin xyz="0 0 0.4" rpy="0 0 0" />
+  <VLP-16 parent="base_link" name="velodyne" topic="/velodyne_points" hz="10" samples="1800" max_range="3.0">
+    <origin xyz="0 0 0.3" rpy="0 0 0" />
   </VLP-16>
   <!-- VHDL-32E -->

Commit message: save trajectory

File: urdf/jackal_velodyne.urdf.xacro (robot description, xacro)
@@ -1,4 +1,5 @@
 <?xml version="1.0"?>
-<robot name="jackal" xmlns:xacro="http://www.ros.org/wiki/xacro">
+<robot name="jackal"
+  xmlns:xacro="http://www.ros.org/wiki/xacro">
   <xacro:property name="PI" value="3.1415926535897931" />
   <xacro:property name="wheelbase" value="0.262" />
@@ -13,8 +14,16 @@
   <xacro:property name="dummy_inertia" value="1e-09"/>
   <xacro:property name="mount_spacing" value="0.120" />
-  <material name="dark_grey"><color rgba="0.2 0.2 0.2 1.0" /></material>
-  <material name="light_grey"><color rgba="0.4 0.4 0.4 1.0" /></material>
-  <material name="yellow"><color rgba="0.8 0.8 0.0 1.0" /></material>
-  <material name="black"><color rgba="0.15 0.15 0.15 1.0" /></material>
+  <material name="dark_grey">
+    <color rgba="0.2 0.2 0.2 1.0" />
+  </material>
+  <material name="light_grey">
+    <color rgba="0.4 0.4 0.4 1.0" />
+  </material>
+  <material name="yellow">
+    <color rgba="0.8 0.8 0.0 1.0" />
+  </material>
+  <material name="black">
+    <color rgba="0.15 0.15 0.15 1.0" />
+  </material>
   <xacro:macro name="wheel" params="prefix *joint_pose">
     <link name="${prefix}_wheel_link">
@@ -35,8 +44,5 @@
         <origin xyz="0 0 0" rpy="0 0 0"/>
         <mass value="0.477"/>
-        <inertia
-          ixx="0.0013" ixy="0" ixz="0"
-          iyy="0.0024" iyz="0"
-          izz="0.0013"/>
+        <inertia ixx="0.0013" ixy="0" ixz="0" iyy="0.0024" iyz="0" izz="0.0013"/>
       </inertial>
     </link>
@@ -99,9 +105,6 @@
       <mass value="16.523"/>
       <!-- Moments of inertia: ( chassis without wheels ) -->
-      <inertia
-        ixx="0.3136" ixy="-0.0008" ixz="0.0164"
-        iyy="0.3922" iyz="-0.0009"
-        izz="0.4485"/>
-      </inertial>
+      <inertia ixx="0.3136" ixy="-0.0008" ixz="0.0164" iyy="0.3922" iyz="-0.0009" izz="0.4485"/>
+    </inertial>
   </link>
   <link name="fenders_link">
@@ -160,10 +163,4 @@
     <origin xyz="${-mount_spacing} 0 0" />
   </joint>
-  <link name="front_mount"></link>
-  <joint name="front_mount_joint" type="fixed">
-    <parent link="mid_mount" />
-    <child link="front_mount" />
-    <origin xyz="${mount_spacing} 0 0" />
-  </joint>
   <!-- Bring in simulation data for Gazebo. -->
   <xacro:include filename="$(find jackal_description)/urdf/jackal.gazebo" />
@@ -178,9 +175,9 @@
   <!-- VLP-16 -->
   <xacro:include filename="$(find velodyne_description)/urdf/VLP-16.urdf.xacro"/>
-  <VLP-16 parent="base_link" name="velodyne" topic="/velodyne_points" hz="10" samples="1800" max_range="3.0">
+  <VLP-16 parent="base_link" name="velodyne" topic="/velodyne_points" hz="10" samples="1800" max_range="3.0" gpu="true">
     <origin xyz="0 0 0.3" rpy="0 0 0" />
   </VLP-16>
   <!-- VHDL-32E -->
-<!--   <xacro:include filename="$(find velodyne_description)/urdf/HDL-32E.urdf.xacro"/>
+  <!--   <xacro:include filename="$(find velodyne_description)/urdf/HDL-32E.urdf.xacro"/>
   <HDL-32E parent="base_link" name="velodyne_2" topic="/velodyne_points_2" hz="10" samples="1800">
     <origin xyz="0 0 0.6" rpy="0 0 0" />

Commit message: Fix front_mount

File: urdf/jackal_velodyne.urdf.xacro (robot description, xacro)
@@ -163,4 +163,10 @@
     <origin xyz="${-mount_spacing} 0 0" />
   </joint>
+  <link name="front_mount"></link>
+  <joint name="front_mount_joint" type="fixed">
+    <parent link="mid_mount" />
+    <child link="front_mount" />
+    <origin xyz="${mount_spacing} 0 0" />
+  </joint>
   <!-- Bring in simulation data for Gazebo. -->
   <xacro:include filename="$(find jackal_description)/urdf/jackal.gazebo" />

Commit message: update rviz config

File: urdf/jackal_velodyne.urdf.xacro (robot description, xacro)
@@ -179,5 +179,5 @@
   <xacro:include filename="$(find velodyne_description)/urdf/VLP-16.urdf.xacro"/>
   <VLP-16 parent="base_link" name="velodyne" topic="/velodyne_points" hz="10" samples="180">
-    <origin xyz="0 0 0.4" rpy="0 0 0" />
+    <origin xyz="0 0 0.3" rpy="0 0 0" />
   </VLP-16>
   <!-- VHDL-32E -->

Commit message: adjust velodyne height

File: urdf/jackal_velodyne.urdf.xacro (robot description, xacro)
@@ -179,5 +179,5 @@
   <xacro:include filename="$(find velodyne_description)/urdf/VLP-16.urdf.xacro"/>
   <VLP-16 parent="base_link" name="velodyne" topic="/velodyne_points" hz="10" samples="1800" gpu="false">
-    <origin xyz="0 0 0.3" rpy="0 0 0" />
+    <origin xyz="0 0 0.4" rpy="0 0 0" />
   </VLP-16>
   <!-- VHDL-32E -->
